Commit message: add first left arm control

File: urdf/eddie.urdf (robot description, URDF)
Before this commit: robot freddy, 57 links, 56 joints
Links:
- link kinova_left_bracelet_link: mass 0.525 -> 0.975

Commit message: add  target pose offset wrt ee for left arm

File: urdf/eddie.urdf (robot description, URDF)
Before this commit: robot freddy, 57 links, 56 joints
Links:
- link kinova_left_bracelet_link: mass 1.425 -> 0.500
