Commit message: - changed interface.cpp to use the eddie_description package - added a new launch file for real robot - removed some old urdf files, launch files, and meshes - kept the initial eddie.urdf file (although it is not being used currently)

File: urdf/eddie.urdf (robot description, URDF)
Before this commit: robot eddie_base_with_wheels, 63 links, 62 joints
Links:
- removed link eddie_base_footprint
- removed link eddie_base_link
- removed link eddie_front_left_left_wheel_link
- removed link eddie_front_left_right_wheel_link
- removed link eddie_front_left_struct_attachment_link
- removed link eddie_front_left_struct_link
- removed link eddie_front_right_left_wheel_link
- removed link eddie_front_right_right_wheel_link
- removed link eddie_front_right_struct_attachment_link
- removed link eddie_front_right_struct_link
- removed link eddie_left_arm_attachment_link
- removed link eddie_left_arm_base_link
- removed link eddie_left_arm_bracelet_link
- removed link eddie_left_arm_camera_color_frame
- removed link eddie_left_arm_camera_depth_frame
- removed link eddie_left_arm_camera_link
- removed link eddie_left_arm_end_effector_link
- removed link eddie_left_arm_forearm_link
- removed link eddie_left_arm_half_arm_1_link
- removed link eddie_left_arm_half_arm_2_link
- removed link eddie_left_arm_robotiq_85_base_link
- removed link eddie_left_arm_robotiq_85_left_finger_link
- removed link eddie_left_arm_robotiq_85_left_finger_tip_link
- removed link eddie_left_arm_robotiq_85_left_inner_knuckle_link
- removed link eddie_left_arm_robotiq_85_left_knuckle_link
- removed link eddie_left_arm_robotiq_85_right_finger_link
- removed link eddie_left_arm_robotiq_85_right_finger_tip_link
- removed link eddie_left_arm_robotiq_85_right_inner_knuckle_link
- removed link eddie_left_arm_robotiq_85_right_knuckle_link
- removed link eddie_left_arm_shoulder_link
- removed link eddie_left_arm_spherical_wrist_1_link
- removed link eddie_left_arm_spherical_wrist_2_link
- removed link eddie_rear_left_left_wheel_link
- removed link eddie_rear_left_right_wheel_link
- removed link eddie_rear_left_struct_attachment_link
- removed link eddie_rear_left_struct_link
- removed link eddie_rear_right_left_wheel_link
- removed link eddie_rear_right_right_wheel_link
- removed link eddie_rear_right_struct_attachment_link
- removed link eddie_rear_right_struct_link
- removed link eddie_right_arm_attachment_link
- removed link eddie_right_arm_base_link
- removed link eddie_right_arm_bracelet_link
- removed link eddie_right_arm_camera_color_frame
- removed link eddie_right_arm_camera_depth_frame
- removed link eddie_right_arm_camera_link
- removed link eddie_right_arm_end_effector_link
- removed link eddie_right_arm_forearm_link
- removed link eddie_right_arm_half_arm_1_link
- removed link eddie_right_arm_half_arm_2_link
- removed link eddie_right_arm_robotiq_85_base_link
- removed link eddie_right_arm_robotiq_85_left_finger_link
- removed link eddie_right_arm_robotiq_85_left_finger_tip_link
- removed link eddie_right_arm_robotiq_85_left_inner_knuckle_link
- removed link eddie_right_arm_robotiq_85_left_knuckle_link
- removed link eddie_right_arm_robotiq_85_right_finger_link
- removed link eddie_right_arm_robotiq_85_right_finger_tip_link
- removed link eddie_right_arm_robotiq_85_right_inner_knuckle_link
- removed link eddie_right_arm_robotiq_85_right_knuckle_link
- removed link eddie_right_arm_shoulder_link
- removed link eddie_right_arm_spherical_wrist_1_link
- removed link eddie_right_arm_spherical_wrist_2_link
- removed link eddie_torso_link
- added link base_laser_back_link, mass 0.16; collision mesh filename=package://freddy_base_description/meshes/sensors/hokuyo_con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; visual mesh filename=package://freddy_base_description/meshes/sensors/hokuyo.dae
- added link base_laser_front_link, mass 0.16; collision mesh filename=package://freddy_base_description/meshes/sensors/hokuyo_con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; visual mesh filename=package://freddy_base_description/meshes/sensors/hokuyo.dae
- added link base_link
- added link freddy_base_link, mass 40.0; collision box size=0.635 0.582 0.1; collision box size=0.635 0.582 0.12
- added link freddy_torso_link, mass 40.0; collision box size=0.19 0.4 0.3; visual box size=0.19 0.4 0.3
- added link freddy_torso_shoulder_left_arm_attach_link
- added link freddy_torso_shoulder_left_link, mass 40.0; collision box size=0.02 0.2 0.2; visual box size=0.02 0.2 0.2
- added link freddy_torso_shoulder_right_arm_attach_link
- added link freddy_torso_shoulder_right_link, mass 40.0; collision box size=0.02 0.2 0.2; visual box size=0.02 0.2 0.2
- added link kinova_left_base_link, mass 1.697; collision mesh filename=file:///home/batsy/freddy/install/kortex_description/share/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; visual mesh filename=file:///home/batsy/freddy/install/kortex_description/share/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
- added link kinova_left_bracelet_link, mass 0.500; collision mesh filename=file:///home/batsy/freddy/install/kortex_description/share/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; visual mesh filename=file:///home/batsy/freddy/install/kortex_description/share/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
- added link kinova_left_camera_color_frame
- added link kinova_left_camera_depth_frame
- added link kinova_left_camera_link
- added link kinova_left_end_effector_link
- added link kinova_left_forearm_link, mass 0.9302; collision mesh filename=file:///home/batsy/freddy/install/kortex_description/share/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; visual mesh filename=file:///home/batsy/freddy/install/kortex_description/share/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
- added link kinova_left_grasp_link
- added link kinova_left_half_arm_1_link, mass 1.1636; collision mesh filename=file:///home/batsy/freddy/install/kortex_description/share/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; visual mesh filename=file:///home/batsy/freddy/install/kortex_description/share/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
- added link kinova_left_half_arm_2_link, mass 1.1636; collision mesh filename=file:///home/batsy/freddy/install/kortex_description/share/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; visual mesh filename=file:///home/batsy/freddy/install/kortex_description/share/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
- added link kinova_left_robotiq_85_base_link, mass 6.6320197e-01; collision mesh filename=file:///home/batsy/freddy/install/robotiq_description/share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; visual mesh filename=file:///home/batsy/freddy/install/robotiq_description/share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
- added link kinova_left_robotiq_85_left_finger_link, mass 4.260376752e-02; collision mesh filename=file:///home/batsy/freddy/install/robotiq_description/share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; visual mesh filename=file:///home/batsy/freddy/install/robotiq_description/share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
- added link kinova_left_robotiq_85_left_finger_tip_link, mass 4.268588744e-02; collision mesh filename=file:///home/batsy/freddy/install/robotiq_description/share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; visual mesh filename=file:///home/batsy/freddy/install/robotiq_description/share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
- added link kinova_left_robotiq_85_left_inner_knuckle_link, mass 2.969376448e-02; collision mesh filename=file:///home/batsy/freddy/install/robotiq_description/share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; visual mesh filename=file:///home/batsy/freddy/install/robotiq_description/share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
- added link kinova_left_robotiq_85_left_knuckle_link, mass 1.384773208e-02; collision mesh filename=file:///home/batsy/freddy/install/robotiq_description/share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; visual mesh filename=file:///home/batsy/freddy/install/robotiq_description/share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
- added link kinova_left_robotiq_85_right_finger_link, mass 4.260376752000000e-02; collision mesh filename=file:///home/batsy/freddy/install/robotiq_description/share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; visual mesh filename=file:///home/batsy/freddy/install/robotiq_description/share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
- added link kinova_left_robotiq_85_right_finger_tip_link, mass 4.268588744e-02; collision mesh filename=file:///home/batsy/freddy/install/robotiq_description/share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; visual mesh filename=file:///home/batsy/freddy/install/robotiq_description/share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
- added link kinova_left_robotiq_85_right_inner_knuckle_link, mass 2.969376448e-02; collision mesh filename=file:///home/batsy/freddy/install/robotiq_description/share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; visual mesh filename=file:///home/batsy/freddy/install/robotiq_description/share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
- added link kinova_left_robotiq_85_right_knuckle_link, mass 1.384773208e-02; collision mesh filename=file:///home/batsy/freddy/install/robotiq_description/share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; visual mesh filename=file:///home/batsy/freddy/install/robotiq_description/share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
- added link kinova_left_shoulder_link, mass 1.3773; collision mesh filename=file:///home/batsy/freddy/install/kortex_description/share/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; visual mesh filename=file:///home/batsy/freddy/install/kortex_description/share/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
- added link kinova_left_spherical_wrist_1_link, mass 0.6781; collision mesh filename=file:///home/batsy/freddy/install/kortex_description/share/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; visual mesh filename=file:///home/batsy/freddy/install/kortex_description/share/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
- added link kinova_left_spherical_wrist_2_link, mass 0.6781; collision mesh filename=file:///home/batsy/freddy/install/kortex_description/share/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; visual mesh filename=file:///home/batsy/freddy/install/kortex_description/share/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
- added link kinova_right_base_link, mass 1.697; collision mesh filename=file:///home/batsy/freddy/install/kortex_description/share/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; visual mesh filename=file:///home/batsy/freddy/install/kortex_description/share/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
- added link kinova_right_bracelet_link, mass 0.500; collision mesh filename=file:///home/batsy/freddy/install/kortex_description/share/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; visual mesh filename=file:///home/batsy/freddy/install/kortex_description/share/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
- added link kinova_right_camera_color_frame
- added link kinova_right_camera_depth_frame
- added link kinova_right_camera_link
- added link kinova_right_end_effector_link
- added link kinova_right_forearm_link, mass 0.9302; collision mesh filename=file:///home/batsy/freddy/install/kortex_description/share/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; visual mesh filename=file:///home/batsy/freddy/install/kortex_description/share/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
- added link kinova_right_grasp_link
- added link kinova_right_half_arm_1_link, mass 1.1636; collision mesh filename=file:///home/batsy/freddy/install/kortex_description/share/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; visual mesh filename=file:///home/batsy/freddy/install/kortex_description/share/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
- added link kinova_right_half_arm_2_link, mass 1.1636; collision mesh filename=file:///home/batsy/freddy/install/kortex_description/share/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; visual mesh filename=file:///home/batsy/freddy/install/kortex_description/share/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
- added link kinova_right_robotiq_85_base_link, mass 6.6320197e-01; collision mesh filename=file:///home/batsy/freddy/install/robotiq_description/share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; visual mesh filename=file:///home/batsy/freddy/install/robotiq_description/share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
- added link kinova_right_robotiq_85_left_finger_link, mass 4.260376752e-02; collision mesh filename=file:///home/batsy/freddy/install/robotiq_description/share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; visual mesh filename=file:///home/batsy/freddy/install/robotiq_description/share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
- added link kinova_right_robotiq_85_left_finger_tip_link, mass 4.268588744e-02; collision mesh filename=file:///home/batsy/freddy/install/robotiq_description/share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; visual mesh filename=file:///home/batsy/freddy/install/robotiq_description/share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
- added link kinova_right_robotiq_85_left_inner_knuckle_link, mass 2.969376448e-02; collision mesh filename=file:///home/batsy/freddy/install/robotiq_description/share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; visual mesh filename=file:///home/batsy/freddy/install/robotiq_description/share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
- added link kinova_right_robotiq_85_left_knuckle_link, mass 1.384773208e-02; collision mesh filename=file:///home/batsy/freddy/install/robotiq_description/share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; visual mesh filename=file:///home/batsy/freddy/install/robotiq_description/share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
- added link kinova_right_robotiq_85_right_finger_link, mass 4.260376752000000e-02; collision mesh filename=file:///home/batsy/freddy/install/robotiq_description/share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; visual mesh filename=file:///home/batsy/freddy/install/robotiq_description/share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
- added link kinova_right_robotiq_85_right_finger_tip_link, mass 4.268588744e-02; collision mesh filename=file:///home/batsy/freddy/install/robotiq_description/share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; visual mesh filename=file:///home/batsy/freddy/install/robotiq_description/share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
- added link kinova_right_robotiq_85_right_inner_knuckle_link, mass 2.969376448e-02; collision mesh filename=file:///home/batsy/freddy/install/robotiq_description/share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; visual mesh filename=file:///home/batsy/freddy/install/robotiq_description/share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
- added link kinova_right_robotiq_85_right_knuckle_link, mass 1.384773208e-02; collision mesh filename=file:///home/batsy/freddy/install/robotiq_description/share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; visual mesh filename=file:///home/batsy/freddy/install/robotiq_description/share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
- added link kinova_right_shoulder_link, mass 1.3773; collision mesh filename=file:///home/batsy/freddy/install/kortex_description/share/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; visual mesh filename=file:///home/batsy/freddy/install/kortex_description/share/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
- added link kinova_right_spherical_wrist_1_link, mass 0.6781; collision mesh filename=file:///home/batsy/freddy/install/kortex_description/share/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; visual mesh filename=file:///home/batsy/freddy/install/kortex_description/share/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
- added link kinova_right_spherical_wrist_2_link, mass 0.6781; collision mesh filename=file:///home/batsy/freddy/install/kortex_description/share/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; visual mesh filename=file:///home/batsy/freddy/install/kortex_description/share/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
- added link left_back_wheel_link, mass 1.0; collision sphere radius=0.05; visual sphere radius=0.05
- added link left_front_wheel_link, mass 1.0; collision sphere radius=0.05; visual sphere radius=0.05
- added link right_back_wheel_link, mass 1.0; collision sphere radius=0.05; visual sphere radius=0.05
- added link right_front_wheel_link, mass 1.0; collision sphere radius=0.05; visual sphere radius=0.05
Joints:
- removed joint eddie_base_footprint_joint
- removed joint eddie_base_torso_joint
- removed joint eddie_front_left_eddie_front_left_left_wheel_joint
- removed joint eddie_front_left_eddie_front_left_right_wheel_joint
- removed joint eddie_front_left_joint
- removed joint eddie_front_left_struct_to_attachment_joint
- removed joint eddie_front_right_eddie_front_right_left_wheel_joint
- removed joint eddie_front_right_eddie_front_right_right_wheel_joint
- removed joint eddie_front_right_joint
- removed joint eddie_front_right_struct_to_attachment_joint
- removed joint eddie_left_arm_attachment_joint
- removed joint eddie_left_arm_base_joint
- removed joint eddie_left_arm_camera_module
- removed joint eddie_left_arm_color_module
- removed joint eddie_left_arm_depth_module
- removed joint eddie_left_arm_end_effector
- removed joint eddie_left_arm_joint_1
- removed joint eddie_left_arm_joint_2
- removed joint eddie_left_arm_joint_3
- removed joint eddie_left_arm_joint_4
- removed joint eddie_left_arm_joint_5
- removed joint eddie_left_arm_joint_6
- removed joint eddie_left_arm_joint_7
- removed joint eddie_left_arm_robotiq_85_base_joint
- removed joint eddie_left_arm_robotiq_85_left_finger_joint
- removed joint eddie_left_arm_robotiq_85_left_finger_tip_joint
- removed joint eddie_left_arm_robotiq_85_left_inner_knuckle_joint
- removed joint eddie_left_arm_robotiq_85_left_knuckle_joint
- removed joint eddie_left_arm_robotiq_85_right_finger_joint
- removed joint eddie_left_arm_robotiq_85_right_finger_tip_joint
- removed joint eddie_left_arm_robotiq_85_right_inner_knuckle_joint
- removed joint eddie_left_arm_robotiq_85_right_knuckle_joint
- removed joint eddie_rear_left_eddie_rear_left_left_wheel_joint
- removed joint eddie_rear_left_eddie_rear_left_right_wheel_joint
- removed joint eddie_rear_left_joint
- removed joint eddie_rear_left_struct_to_attachment_joint
- removed joint eddie_rear_right_eddie_rear_right_left_wheel_joint
- removed joint eddie_rear_right_eddie_rear_right_right_wheel_joint
- removed joint eddie_rear_right_joint
- removed joint eddie_rear_right_struct_to_attachment_joint
- removed joint eddie_right_arm_attachment_joint
- removed joint eddie_right_arm_base_joint
- removed joint eddie_right_arm_camera_module
- removed joint eddie_right_arm_color_module
- removed joint eddie_right_arm_depth_module
- removed joint eddie_right_arm_end_effector
- removed joint eddie_right_arm_joint_1
- removed joint eddie_right_arm_joint_2
- removed joint eddie_right_arm_joint_3
- removed joint eddie_right_arm_joint_4
- removed joint eddie_right_arm_joint_5
- removed joint eddie_right_arm_joint_6
- removed joint eddie_right_arm_joint_7
- removed joint eddie_right_arm_robotiq_85_base_joint
- removed joint eddie_right_arm_robotiq_85_left_finger_joint
- removed joint eddie_right_arm_robotiq_85_left_finger_tip_joint
- removed joint eddie_right_arm_robotiq_85_left_inner_knuckle_joint
- removed joint eddie_right_arm_robotiq_85_left_knuckle_joint
- removed joint eddie_right_arm_robotiq_85_right_finger_joint
- removed joint eddie_right_arm_robotiq_85_right_finger_tip_joint
- removed joint eddie_right_arm_robotiq_85_right_inner_knuckle_joint
- removed joint eddie_right_arm_robotiq_85_right_knuckle_joint
- added joint base_laser_back_joint: type fixed, parent freddy_base_link, child base_laser_back_link, origin xyz=-0.26 0.24 0.25 rpy=3.141592653589793 0 2.356194490192345, axis 0 1 0
- added joint base_laser_front_joint: type fixed, parent freddy_base_link, child base_laser_front_link, origin xyz=0.26 -0.24 0.25 rpy=3.141592653589793 0 -0.7853981633974483, axis 0 1 0
- added joint freddy_base_joint: type fixed, parent base_link, child freddy_base_link, origin xyz=0.0 0.0 0.0 rpy=0.0 0.0 0.0
- added joint freddy_torso_joint: type fixed, parent base_link, child freddy_torso_link, origin xyz=-0.20249999999999999 0 0.37 rpy=0 0 0
- added joint freddy_torso_shoulder_left_arm_joint: type fixed, parent freddy_torso_shoulder_left_link, child freddy_torso_shoulder_left_arm_attach_link, origin xyz=0 0.1 0.1 rpy=3.14159 -1.5708 0
- added joint freddy_torso_shoulder_left_joint: type fixed, parent freddy_torso_link, child freddy_torso_shoulder_left_link, origin xyz=0.085 0 0.27 rpy=0. 0.1309 0.7853982
- added joint freddy_torso_shoulder_right_arm_joint: type fixed, parent freddy_torso_shoulder_right_link, child freddy_torso_shoulder_right_arm_attach_link, origin xyz=0 -0.1 0.1 rpy=3.14159 -1.5708 0
- added joint freddy_torso_shoulder_right_joint: type fixed, parent freddy_torso_link, child freddy_torso_shoulder_right_link, origin xyz=0.085 0 0.27 rpy=0 0.1309 -0.7853982
- added joint kinova_left_base_joint: type fixed, parent freddy_torso_shoulder_left_arm_attach_link, child kinova_left_base_link, origin xyz=0 0 0 rpy=0 0 0
- added joint kinova_left_camera_module: type fixed, parent kinova_left_end_effector_link, child kinova_left_camera_link, origin xyz=0 0.05639 -0.00305 rpy=3.141592653589793 3.141592653589793 0
- added joint kinova_left_color_module: type fixed, parent kinova_left_end_effector_link, child kinova_left_camera_color_frame, origin xyz=0 0.05639 -0.00305 rpy=3.141592653589793 3.141592653589793 0
- added joint kinova_left_depth_module: type fixed, parent kinova_left_end_effector_link, child kinova_left_camera_depth_frame, origin xyz=0.0275 0.066 -0.00305 rpy=3.141592653589793 3.141592653589793 0
- added joint kinova_left_end_effector: type fixed, parent kinova_left_bracelet_link, child kinova_left_end_effector_link, origin xyz=0 0 -0.0615250000000001 rpy=3.14159265358979 1.09937075168372E-32 0, axis 0 0 0
- added joint kinova_left_grasp_link_joint: type fixed, parent kinova_left_robotiq_85_base_link, child kinova_left_grasp_link, origin xyz=0 0 0.15 rpy=0 0 0
- added joint kinova_left_joint_1: type continuous, parent kinova_left_base_link, child kinova_left_shoulder_link, origin xyz=0 0 0.15643 rpy=3.1416 2.7629E-18 -4.9305E-36, axis 0 0 1, limit effort=39 velocity=1.3963
- added joint kinova_left_joint_2: type revolute, parent kinova_left_shoulder_link, child kinova_left_half_arm_1_link, origin xyz=0 0.005375 -0.12838 rpy=1.5708 2.1343E-17 -1.1102E-16, axis 0 0 1, limit lower=-2.41 upper=2.41 effort=39 velocity=1.3963
- added joint kinova_left_joint_3: type continuous, parent kinova_left_half_arm_1_link, child kinova_left_half_arm_2_link, origin xyz=0 -0.21038 -0.006375 rpy=-1.5708 1.2326E-32 -2.9122E-16, axis 0 0 1, limit effort=39 velocity=1.3963
- added joint kinova_left_joint_4: type revolute, parent kinova_left_half_arm_2_link, child kinova_left_forearm_link, origin xyz=0 0.006375 -0.21038 rpy=1.5708 -6.6954E-17 -1.6653E-16, axis 0 0 1, limit lower=-2.66 upper=2.66 effort=39 velocity=1.3963
- added joint kinova_left_joint_5: type continuous, parent kinova_left_forearm_link, child kinova_left_spherical_wrist_1_link, origin xyz=0 -0.20843 -0.006375 rpy=-1.5708 2.2204E-16 -6.373E-17, axis 0 0 1, limit effort=9 velocity=1.2218
- added joint kinova_left_joint_6: type revolute, parent kinova_left_spherical_wrist_1_link, child kinova_left_spherical_wrist_2_link, origin xyz=0 0.00017505 -0.10593 rpy=1.5708 9.2076E-28 -8.2157E-15, axis 0 0 1, limit lower=-2.23 upper=2.23 effort=9 velocity=1.2218
- added joint kinova_left_joint_7: type continuous, parent kinova_left_spherical_wrist_2_link, child kinova_left_bracelet_link, origin xyz=0 -0.10593 -0.00017505 rpy=-1.5708 -5.5511E-17 9.6396E-17, axis 0 0 1, limit effort=9 velocity=1.2218
- added joint kinova_left_robotiq_85_base_joint: type fixed, parent kinova_left_end_effector_link, child kinova_left_robotiq_85_base_link, origin xyz=0 0 0 rpy=0 0 0
- added joint kinova_left_robotiq_85_left_finger_joint: type fixed, parent kinova_left_robotiq_85_left_knuckle_link, child kinova_left_robotiq_85_left_finger_link, origin xyz=0.03152616 0.0 -0.00376347 rpy=0 0 0
- added joint kinova_left_robotiq_85_left_finger_tip_joint: type continuous, parent kinova_left_robotiq_85_left_finger_link, child kinova_left_robotiq_85_left_finger_tip_link, origin xyz=0.00563134 0.0 0.04718515 rpy=0 0 0, axis 0 -1 0, mimic joint=kinova_left_robotiq_85_left_knuckle_joint multiplier=-1
- added joint kinova_left_robotiq_85_left_inner_knuckle_joint: type continuous, parent kinova_left_robotiq_85_base_link, child kinova_left_robotiq_85_left_inner_knuckle_link, origin xyz=0.0127 0.0 0.06142 rpy=0 0 0, axis 0 -1 0, mimic joint=kinova_left_robotiq_85_left_knuckle_joint
- added joint kinova_left_robotiq_85_left_knuckle_joint: type revolute, parent kinova_left_robotiq_85_base_link, child kinova_left_robotiq_85_left_knuckle_link, origin xyz=0.03060114 0.0 0.05490452 rpy=0 0 0, axis 0 -1 0, limit lower=0.0 upper=0.8 effort=50 velocity=0.5
- added joint kinova_left_robotiq_85_right_finger_joint: type fixed, parent kinova_left_robotiq_85_right_knuckle_link, child kinova_left_robotiq_85_right_finger_link, origin xyz=-0.03152616 0.0 -0.00376347 rpy=0 0 0
- added joint kinova_left_robotiq_85_right_finger_tip_joint: type continuous, parent kinova_left_robotiq_85_right_finger_link, child kinova_left_robotiq_85_right_finger_tip_link, origin xyz=-0.00563134 0.0 0.04718515 rpy=0 0 0, axis 0 -1 0, mimic joint=kinova_left_robotiq_85_left_knuckle_joint
- added joint kinova_left_robotiq_85_right_inner_knuckle_joint: type continuous, parent kinova_left_robotiq_85_base_link, child kinova_left_robotiq_85_right_inner_knuckle_link, origin xyz=-0.0127 0.0 0.06142 rpy=0 0 0, axis 0 -1 0, mimic joint=kinova_left_robotiq_85_left_knuckle_joint multiplier=-1
- added joint kinova_left_robotiq_85_right_knuckle_joint: type revolute, parent kinova_left_robotiq_85_base_link, child kinova_left_robotiq_85_right_knuckle_link, origin xyz=-0.03060114 0.0 0.05490452 rpy=0 0 0, axis 0 -1 0, limit lower=-0.8 upper=0.0 effort=50 velocity=0.5, mimic joint=kinova_left_robotiq_85_left_knuckle_joint multiplier=-1
- added joint kinova_right_base_joint: type fixed, parent freddy_torso_shoulder_right_arm_attach_link, child kinova_right_base_link, origin xyz=0 0 0 rpy=0 0 0
- added joint kinova_right_camera_module: type fixed, parent kinova_right_end_effector_link, child kinova_right_camera_link, origin xyz=0 0.05639 -0.00305 rpy=3.141592653589793 3.141592653589793 0
- added joint kinova_right_color_module: type fixed, parent kinova_right_end_effector_link, child kinova_right_camera_color_frame, origin xyz=0 0.05639 -0.00305 rpy=3.141592653589793 3.141592653589793 0
- added joint kinova_right_depth_module: type fixed, parent kinova_right_end_effector_link, child kinova_right_camera_depth_frame, origin xyz=0.0275 0.066 -0.00305 rpy=3.141592653589793 3.141592653589793 0
- added joint kinova_right_end_effector: type fixed, parent kinova_right_bracelet_link, child kinova_right_end_effector_link, origin xyz=0 0 -0.0615250000000001 rpy=3.14159265358979 1.09937075168372E-32 0, axis 0 0 0
- added joint kinova_right_grasp_link_joint: type fixed, parent kinova_right_robotiq_85_base_link, child kinova_right_grasp_link, origin xyz=0 0 0.15 rpy=0 0 0
- added joint kinova_right_joint_1: type continuous, parent kinova_right_base_link, child kinova_right_shoulder_link, origin xyz=0 0 0.15643 rpy=3.1416 2.7629E-18 -4.9305E-36, axis 0 0 1, limit effort=39 velocity=1.3963
- added joint kinova_right_joint_2: type revolute, parent kinova_right_shoulder_link, child kinova_right_half_arm_1_link, origin xyz=0 0.005375 -0.12838 rpy=1.5708 2.1343E-17 -1.1102E-16, axis 0 0 1, limit lower=-2.41 upper=2.41 effort=39 velocity=1.3963
- added joint kinova_right_joint_3: type continuous, parent kinova_right_half_arm_1_link, child kinova_right_half_arm_2_link, origin xyz=0 -0.21038 -0.006375 rpy=-1.5708 1.2326E-32 -2.9122E-16, axis 0 0 1, limit effort=39 velocity=1.3963
- added joint kinova_right_joint_4: type revolute, parent kinova_right_half_arm_2_link, child kinova_right_forearm_link, origin xyz=0 0.006375 -0.21038 rpy=1.5708 -6.6954E-17 -1.6653E-16, axis 0 0 1, limit lower=-2.66 upper=2.66 effort=39 velocity=1.3963
- added joint kinova_right_joint_5: type continuous, parent kinova_right_forearm_link, child kinova_right_spherical_wrist_1_link, origin xyz=0 -0.20843 -0.006375 rpy=-1.5708 2.2204E-16 -6.373E-17, axis 0 0 1, limit effort=9 velocity=1.2218
- added joint kinova_right_joint_6: type revolute, parent kinova_right_spherical_wrist_1_link, child kinova_right_spherical_wrist_2_link, origin xyz=0 0.00017505 -0.10593 rpy=1.5708 9.2076E-28 -8.2157E-15, axis 0 0 1, limit lower=-2.23 upper=2.23 effort=9 velocity=1.2218
- added joint kinova_right_joint_7: type continuous, parent kinova_right_spherical_wrist_2_link, child kinova_right_bracelet_link, origin xyz=0 -0.10593 -0.00017505 rpy=-1.5708 -5.5511E-17 9.6396E-17, axis 0 0 1, limit effort=9 velocity=1.2218
- added joint kinova_right_robotiq_85_base_joint: type fixed, parent kinova_right_end_effector_link, child kinova_right_robotiq_85_base_link, origin xyz=0 0 0 rpy=0 0 0
- added joint kinova_right_robotiq_85_left_finger_joint: type fixed, parent kinova_right_robotiq_85_left_knuckle_link, child kinova_right_robotiq_85_left_finger_link, origin xyz=0.03152616 0.0 -0.00376347 rpy=0 0 0
- added joint kinova_right_robotiq_85_left_finger_tip_joint: type continuous, parent kinova_right_robotiq_85_left_finger_link, child kinova_right_robotiq_85_left_finger_tip_link, origin xyz=0.00563134 0.0 0.04718515 rpy=0 0 0, axis 0 -1 0, mimic joint=kinova_right_robotiq_85_left_knuckle_joint multiplier=-1
- added joint kinova_right_robotiq_85_left_inner_knuckle_joint: type continuous, parent kinova_right_robotiq_85_base_link, child kinova_right_robotiq_85_left_inner_knuckle_link, origin xyz=0.0127 0.0 0.06142 rpy=0 0 0, axis 0 -1 0, mimic joint=kinova_right_robotiq_85_left_knuckle_joint
- added joint kinova_right_robotiq_85_left_knuckle_joint: type revolute, parent kinova_right_robotiq_85_base_link, child kinova_right_robotiq_85_left_knuckle_link, origin xyz=0.03060114 0.0 0.05490452 rpy=0 0 0, axis 0 -1 0, limit lower=0.0 upper=0.8 effort=50 velocity=0.5
- added joint kinova_right_robotiq_85_right_finger_joint: type fixed, parent kinova_right_robotiq_85_right_knuckle_link, child kinova_right_robotiq_85_right_finger_link, origin xyz=-0.03152616 0.0 -0.00376347 rpy=0 0 0
- added joint kinova_right_robotiq_85_right_finger_tip_joint: type continuous, parent kinova_right_robotiq_85_right_finger_link, child kinova_right_robotiq_85_right_finger_tip_link, origin xyz=-0.00563134 0.0 0.04718515 rpy=0 0 0, axis 0 -1 0, mimic joint=kinova_right_robotiq_85_left_knuckle_joint
- added joint kinova_right_robotiq_85_right_inner_knuckle_joint: type continuous, parent kinova_right_robotiq_85_base_link, child kinova_right_robotiq_85_right_inner_knuckle_link, origin xyz=-0.0127 0.0 0.06142 rpy=0 0 0, axis 0 -1 0, mimic joint=kinova_right_robotiq_85_left_knuckle_joint multiplier=-1
- added joint kinova_right_robotiq_85_right_knuckle_joint: type revolute, parent kinova_right_robotiq_85_base_link, child kinova_right_robotiq_85_right_knuckle_link, origin xyz=-0.03060114 0.0 0.05490452 rpy=0 0 0, axis 0 -1 0, limit lower=-0.8 upper=0.0 effort=50 velocity=0.5, mimic joint=kinova_right_robotiq_85_left_knuckle_joint multiplier=-1
- added joint left_back_wheel_joint: type fixed, parent freddy_base_link, child left_back_wheel_link, origin xyz=-0.2675                          0.241                          0.05 rpy=0 0 0
- added joint left_front_wheel_joint: type fixed, parent freddy_base_link, child left_front_wheel_link, origin xyz=0.2675                          0.241                          0.05 rpy=0 0 0
- added joint right_back_wheel_joint: type fixed, parent freddy_base_link, child right_back_wheel_link, origin xyz=-0.2675                          -0.241                          0.05 rpy=0 0 0
- added joint right_front_wheel_joint: type fixed, parent freddy_base_link, child right_front_wheel_link, origin xyz=0.2675                          -0.241                          0.05 rpy=0 0 0
