Commit message: fix kdl chain for right arm

File: urdf/eddie.urdf (robot description, URDF)
Before this commit: robot freddy, 57 links, 56 joints
Links:
- removed link base_laser_back_link
- removed link base_laser_front_link
- removed link base_link
- removed link freddy_base_link
- removed link freddy_torso_link
- removed link freddy_torso_shoulder_left_arm_attach_link
- removed link freddy_torso_shoulder_left_link
- removed link freddy_torso_shoulder_right_arm_attach_link
- removed link freddy_torso_shoulder_right_link
- removed link kinova_left_base_link
- removed link kinova_left_bracelet_link
- removed link kinova_left_camera_color_frame
- removed link kinova_left_camera_depth_frame
- removed link kinova_left_camera_link
- removed link kinova_left_end_effector_link
- removed link kinova_left_forearm_link
- removed link kinova_left_grasp_link
- removed link kinova_left_half_arm_1_link
- removed link kinova_left_half_arm_2_link
- removed link kinova_left_robotiq_85_base_link
- removed link kinova_left_robotiq_85_left_finger_link
- removed link kinova_left_robotiq_85_left_finger_tip_link
- removed link kinova_left_robotiq_85_left_inner_knuckle_link
- removed link kinova_left_robotiq_85_left_knuckle_link
- removed link kinova_left_robotiq_85_right_finger_link
- removed link kinova_left_robotiq_85_right_finger_tip_link
- removed link kinova_left_robotiq_85_right_inner_knuckle_link
- removed link kinova_left_robotiq_85_right_knuckle_link
- removed link kinova_left_shoulder_link
- removed link kinova_left_spherical_wrist_1_link
- removed link kinova_left_spherical_wrist_2_link
- removed link kinova_right_base_link
- removed link kinova_right_bracelet_link
- removed link kinova_right_camera_color_frame
- removed link kinova_right_camera_depth_frame
- removed link kinova_right_camera_link
- removed link kinova_right_end_effector_link
- removed link kinova_right_forearm_link
- removed link kinova_right_grasp_link
- removed link kinova_right_half_arm_1_link
- removed link kinova_right_half_arm_2_link
- removed link kinova_right_robotiq_85_base_link
- removed link kinova_right_robotiq_85_left_finger_link
- removed link kinova_right_robotiq_85_left_finger_tip_link
- removed link kinova_right_robotiq_85_left_inner_knuckle_link
- removed link kinova_right_robotiq_85_left_knuckle_link
- removed link kinova_right_robotiq_85_right_finger_link
- removed link kinova_right_robotiq_85_right_finger_tip_link
- removed link kinova_right_robotiq_85_right_inner_knuckle_link
- removed link kinova_right_robotiq_85_right_knuckle_link
- removed link kinova_right_shoulder_link
- removed link kinova_right_spherical_wrist_1_link
- removed link kinova_right_spherical_wrist_2_link
- removed link left_back_wheel_link
- removed link left_front_wheel_link
- removed link right_back_wheel_link
- removed link right_front_wheel_link
- added link eddie_base_footprint
- added link eddie_base_link, mass 76.4377; collision mesh filename=package://eddie_description/meshes/kelo_base.stl; collision mesh filename=package://eddie_description/meshes/kelo_torso.stl
- added link eddie_front_left_drive_attachment_link, mass 0.5; collision mesh filename=package://eddie_description/meshes/kelo_drive_attachments.s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; visual mesh filename=package://eddie_description/meshes/kelo_drive_attachments.s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
- added link eddie_front_left_drive_l_wheel_link, mass 1.563; collision mesh filename=package://eddie_description/meshes/hub_wheel.stl; visual mesh filename=package://eddie_description/meshes/hub_wheel.stl
- added link eddie_front_left_drive_r_wheel_link, mass 1.563; collision mesh filename=package://eddie_description/meshes/hub_wheel.stl; visual mesh filename=package://eddie_description/meshes/hub_wheel.stl
- added link eddie_front_left_drive_struct_link, mass 1.392; collision mesh filename=package://eddie_description/meshes/kelo_drive.stl; visual mesh filename=package://eddie_description/meshes/kelo_drive.stl
- added link eddie_front_right_drive_attachment_link, mass 0.5; collision mesh filename=package://eddie_description/meshes/kelo_drive_attachments.s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; visual mesh filename=package://eddie_description/meshes/kelo_drive_attachments.s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
- added link eddie_front_right_drive_l_wheel_link, mass 1.563; collision mesh filename=package://eddie_description/meshes/hub_wheel.stl; visual mesh filename=package://eddie_description/meshes/hub_wheel.stl
- added link eddie_front_right_drive_r_wheel_link, mass 1.563; collision mesh filename=package://eddie_description/meshes/hub_wheel.stl; visual mesh filename=package://eddie_description/meshes/hub_wheel.stl
- added link eddie_front_right_drive_struct_link, mass 1.392; collision mesh filename=package://eddie_description/meshes/kelo_drive.stl; visual mesh filename=package://eddie_description/meshes/kelo_drive.stl
- added link eddie_front_right_laser_attachment_link
- added link eddie_front_right_laser_link, mass 0.16; collision mesh filename=package://eddie_description/meshes/sensors/hokuyo_convex.dae; visual mesh filename=package://eddie_description/meshes/sensors/hokuyo.dae
- added link eddie_imu_link
- added link eddie_left_arm_attachment_link
- added link eddie_left_arm_base_link, mass 1.697; collision mesh filename=file:///home/bhunecke/r4s/install/kortex_description/share/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; visual mesh filename=file:///home/bhunecke/r4s/install/kortex_description/share/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
- added link eddie_left_arm_bracelet_link, mass 0.5; collision mesh filename=file:///home/bhunecke/r4s/install/kortex_description/share/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; visual mesh filename=file:///home/bhunecke/r4s/install/kortex_description/share/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
- added link eddie_left_arm_camera_color_frame
- added link eddie_left_arm_camera_depth_frame
- added link eddie_left_arm_camera_link
- added link eddie_left_arm_end_effector_link
- added link eddie_left_arm_forearm_link, mass 0.9302; collision mesh filename=file:///home/bhunecke/r4s/install/kortex_description/share/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; visual mesh filename=file:///home/bhunecke/r4s/install/kortex_description/share/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
- added link eddie_left_arm_half_arm_1_link, mass 1.1636; collision mesh filename=file:///home/bhunecke/r4s/install/kortex_description/share/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; visual mesh filename=file:///home/bhunecke/r4s/install/kortex_description/share/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
- added link eddie_left_arm_half_arm_2_link, mass 1.1636; collision mesh filename=file:///home/bhunecke/r4s/install/kortex_description/share/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; visual mesh filename=file:///home/bhunecke/r4s/install/kortex_description/share/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
- added link eddie_left_arm_robotiq_85_base_link, mass 6.6320197e-01; collision mesh filename=package://robotiq_description/meshes/collision/2f_85/roboti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; visual mesh filename=package://robotiq_description/meshes/visual/2f_85/robotiq_b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
- added link eddie_left_arm_robotiq_85_grasp_link
- added link eddie_left_arm_robotiq_85_left_finger_link, mass 4.260376752e-02; collision mesh filename=package://robotiq_description/meshes/collision/2f_85/left_f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; visual mesh filename=package://robotiq_description/meshes/visual/2f_85/left_fing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
- added link eddie_left_arm_robotiq_85_left_finger_tip_link, mass 4.268588744e-02; collision mesh filename=package://robotiq_description/meshes/collision/2f_85/left_f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; visual mesh filename=package://robotiq_description/meshes/visual/2f_85/left_fing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
- added link eddie_left_arm_robotiq_85_left_inner_knuckle_link, mass 2.969376448e-02; collision mesh filename=package://robotiq_description/meshes/collision/2f_85/left_i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; visual mesh filename=package://robotiq_description/meshes/visual/2f_85/left_inne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
- added link eddie_left_arm_robotiq_85_left_knuckle_link, mass 1.384773208e-02; collision mesh filename=package://robotiq_description/meshes/collision/2f_85/left_k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; visual mesh filename=package://robotiq_description/meshes/visual/2f_85/left_knuc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
- added link eddie_left_arm_robotiq_85_right_finger_link, mass 4.260376752000000e-02; collision mesh filename=package://robotiq_description/meshes/collision/2f_85/right_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; visual mesh filename=package://robotiq_description/meshes/visual/2f_85/right_fin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
- added link eddie_left_arm_robotiq_85_right_finger_tip_link, mass 4.268588744e-02; collision mesh filename=package://robotiq_description/meshes/collision/2f_85/right_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; visual mesh filename=package://robotiq_description/meshes/visual/2f_85/right_fin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
- added link eddie_left_arm_robotiq_85_right_inner_knuckle_link, mass 2.969376448e-02; collision mesh filename=package://robotiq_description/meshes/collision/2f_85/right_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; visual mesh filename=package://robotiq_description/meshes/visual/2f_85/right_inn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
- added link eddie_left_arm_robotiq_85_right_knuckle_link, mass 1.384773208e-02; collision mesh filename=package://robotiq_description/meshes/collision/2f_85/right_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; visual mesh filename=package://robotiq_description/meshes/visual/2f_85/right_knu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
- added link eddie_left_arm_shoulder_link, mass 1.3773; collision mesh filename=file:///home/bhunecke/r4s/install/kortex_description/share/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; visual mesh filename=file:///home/bhunecke/r4s/install/kortex_description/share/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
- added link eddie_left_arm_spherical_wrist_1_link, mass 0.6781; collision mesh filename=file:///home/bhunecke/r4s/install/kortex_description/share/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; visual mesh filename=file:///home/bhunecke/r4s/install/kortex_description/share/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
- added link eddie_left_arm_spherical_wrist_2_link, mass 0.6781; collision mesh filename=file:///home/bhunecke/r4s/install/kortex_description/share/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; visual mesh filename=file:///home/bhunecke/r4s/install/kortex_description/share/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
- added link eddie_rear_left_drive_attachment_link, mass 0.5; collision mesh filename=package://eddie_description/meshes/kelo_drive_attachments.s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; visual mesh filename=package://eddie_description/meshes/kelo_drive_attachments.s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
- added link eddie_rear_left_drive_l_wheel_link, mass 1.563; collision mesh filename=package://eddie_description/meshes/hub_wheel.stl; visual mesh filename=package://eddie_description/meshes/hub_wheel.stl
- added link eddie_rear_left_drive_r_wheel_link, mass 1.563; collision mesh filename=package://eddie_description/meshes/hub_wheel.stl; visual mesh filename=package://eddie_description/meshes/hub_wheel.stl
- added link eddie_rear_left_drive_struct_link, mass 1.392; collision mesh filename=package://eddie_description/meshes/kelo_drive.stl; visual mesh filename=package://eddie_description/meshes/kelo_drive.stl
- added link eddie_rear_left_laser_attachment_link
- added link eddie_rear_left_laser_link, mass 0.16; collision mesh filename=package://eddie_description/meshes/sensors/hokuyo_convex.dae; visual mesh filename=package://eddie_description/meshes/sensors/hokuyo.dae
- added link eddie_rear_right_drive_attachment_link, mass 0.5; collision mesh filename=package://eddie_description/meshes/kelo_drive_attachments.s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; visual mesh filename=package://eddie_description/meshes/kelo_drive_attachments.s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
- added link eddie_rear_right_drive_l_wheel_link, mass 1.563; collision mesh filename=package://eddie_description/meshes/hub_wheel.stl; visual mesh filename=package://eddie_description/meshes/hub_wheel.stl
- added link eddie_rear_right_drive_r_wheel_link, mass 1.563; collision mesh filename=package://eddie_description/meshes/hub_wheel.stl; visual mesh filename=package://eddie_description/meshes/hub_wheel.stl
- added link eddie_rear_right_drive_struct_link, mass 1.392; collision mesh filename=package://eddie_description/meshes/kelo_drive.stl; visual mesh filename=package://eddie_description/meshes/kelo_drive.stl
- added link eddie_right_arm_attachment_link
- added link eddie_right_arm_base_link, mass 1.697; collision mesh filename=file:///home/bhunecke/r4s/install/kortex_description/share/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; visual mesh filename=file:///home/bhunecke/r4s/install/kortex_description/share/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
- added link eddie_right_arm_bracelet_link, mass 0.5; collision mesh filename=file:///home/bhunecke/r4s/install/kortex_description/share/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; visual mesh filename=file:///home/bhunecke/r4s/install/kortex_description/share/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
- added link eddie_right_arm_camera_color_frame
- added link eddie_right_arm_camera_depth_frame
- added link eddie_right_arm_camera_link
- added link eddie_right_arm_end_effector_link
- added link eddie_right_arm_forearm_link, mass 0.9302; collision mesh filename=file:///home/bhunecke/r4s/install/kortex_description/share/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; visual mesh filename=file:///home/bhunecke/r4s/install/kortex_description/share/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
- added link eddie_right_arm_ft_sensor_link, mass 0.6; collision cylinder length=0.064 radius=0.0375; visual cylinder length=0.064 radius=0.0375
- added link eddie_right_arm_half_arm_1_link, mass 1.1636; collision mesh filename=file:///home/bhunecke/r4s/install/kortex_description/share/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; visual mesh filename=file:///home/bhunecke/r4s/install/kortex_description/share/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
- added link eddie_right_arm_half_arm_2_link, mass 1.1636; collision mesh filename=file:///home/bhunecke/r4s/install/kortex_description/share/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; visual mesh filename=file:///home/bhunecke/r4s/install/kortex_description/share/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
- added link eddie_right_arm_robotiq_85_base_link, mass 6.6320197e-01; collision mesh filename=package://robotiq_description/meshes/collision/2f_85/roboti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; visual mesh filename=package://robotiq_description/meshes/visual/2f_85/robotiq_b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
- added link eddie_right_arm_robotiq_85_grasp_link
- added link eddie_right_arm_robotiq_85_left_finger_link, mass 4.260376752e-02; collision mesh filename=package://robotiq_description/meshes/collision/2f_85/left_f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; visual mesh filename=package://robotiq_description/meshes/visual/2f_85/left_fing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
- added link eddie_right_arm_robotiq_85_left_finger_tip_link, mass 4.268588744e-02; collision mesh filename=package://robotiq_description/meshes/collision/2f_85/left_f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; visual mesh filename=package://robotiq_description/meshes/visual/2f_85/left_fing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
- added link eddie_right_arm_robotiq_85_left_inner_knuckle_link, mass 2.969376448e-02; collision mesh filename=package://robotiq_description/meshes/collision/2f_85/left_i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; visual mesh filename=package://robotiq_description/meshes/visual/2f_85/left_inne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
- added link eddie_right_arm_robotiq_85_left_knuckle_link, mass 1.384773208e-02; collision mesh filename=package://robotiq_description/meshes/collision/2f_85/left_k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; visual mesh filename=package://robotiq_description/meshes/visual/2f_85/left_knuc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
- added link eddie_right_arm_robotiq_85_right_finger_link, mass 4.260376752000000e-02; collision mesh filename=package://robotiq_description/meshes/collision/2f_85/right_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; visual mesh filename=package://robotiq_description/meshes/visual/2f_85/right_fin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
- added link eddie_right_arm_robotiq_85_right_finger_tip_link, mass 4.268588744e-02; collision mesh filename=package://robotiq_description/meshes/collision/2f_85/right_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; visual mesh filename=package://robotiq_description/meshes/visual/2f_85/right_fin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
- added link eddie_right_arm_robotiq_85_right_inner_knuckle_link, mass 2.969376448e-02; collision mesh filename=package://robotiq_description/meshes/collision/2f_85/right_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; visual mesh filename=package://robotiq_description/meshes/visual/2f_85/right_inn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
- added link eddie_right_arm_robotiq_85_right_knuckle_link, mass 1.384773208e-02; collision mesh filename=package://robotiq_description/meshes/collision/2f_85/right_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; visual mesh filename=package://robotiq_description/meshes/visual/2f_85/right_knu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
- added link eddie_right_arm_shoulder_link, mass 1.3773; collision mesh filename=file:///home/bhunecke/r4s/install/kortex_description/share/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; visual mesh filename=file:///home/bhunecke/r4s/install/kortex_description/share/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
- added link eddie_right_arm_spherical_wrist_1_link, mass 0.6781; collision mesh filename=file:///home/bhunecke/r4s/install/kortex_description/share/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; visual mesh filename=file:///home/bhunecke/r4s/install/kortex_description/share/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
- added link eddie_right_arm_spherical_wrist_2_link, mass 0.6781; collision mesh filename=file:///home/bhunecke/r4s/install/kortex_description/share/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; visual mesh filename=file:///home/bhunecke/r4s/install/kortex_description/share/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
Joints:
- removed joint base_laser_back_joint
- removed joint base_laser_front_joint
- removed joint freddy_base_joint
- removed joint freddy_torso_joint
- removed joint freddy_torso_shoulder_left_arm_joint
- removed joint freddy_torso_shoulder_left_joint
- removed joint freddy_torso_shoulder_right_arm_joint
- removed joint freddy_torso_shoulder_right_joint
- removed joint kinova_left_base_joint
- removed joint kinova_left_camera_module
- removed joint kinova_left_color_module
- removed joint kinova_left_depth_module
- removed joint kinova_left_end_effector
- removed joint kinova_left_grasp_link_joint
- removed joint kinova_left_joint_1
- removed joint kinova_left_joint_2
- removed joint kinova_left_joint_3
- removed joint kinova_left_joint_4
- removed joint kinova_left_joint_5
- removed joint kinova_left_joint_6
- removed joint kinova_left_joint_7
- removed joint kinova_left_robotiq_85_base_joint
- removed joint kinova_left_robotiq_85_left_finger_joint
- removed joint kinova_left_robotiq_85_left_finger_tip_joint
- removed joint kinova_left_robotiq_85_left_inner_knuckle_joint
- removed joint kinova_left_robotiq_85_left_knuckle_joint
- removed joint kinova_left_robotiq_85_right_finger_joint
- removed joint kinova_left_robotiq_85_right_finger_tip_joint
- removed joint kinova_left_robotiq_85_right_inner_knuckle_joint
- removed joint kinova_left_robotiq_85_right_knuckle_joint
- removed joint kinova_right_base_joint
- removed joint kinova_right_camera_module
- removed joint kinova_right_color_module
- removed joint kinova_right_depth_module
- removed joint kinova_right_end_effector
- removed joint kinova_right_grasp_link_joint
- removed joint kinova_right_joint_1
- removed joint kinova_right_joint_2
- removed joint kinova_right_joint_3
- removed joint kinova_right_joint_4
- removed joint kinova_right_joint_5
- removed joint kinova_right_joint_6
- removed joint kinova_right_joint_7
- removed joint kinova_right_robotiq_85_base_joint
- removed joint kinova_right_robotiq_85_left_finger_joint
- removed joint kinova_right_robotiq_85_left_finger_tip_joint
- removed joint kinova_right_robotiq_85_left_inner_knuckle_joint
- removed joint kinova_right_robotiq_85_left_knuckle_joint
- removed joint kinova_right_robotiq_85_right_finger_joint
- removed joint kinova_right_robotiq_85_right_finger_tip_joint
- removed joint kinova_right_robotiq_85_right_inner_knuckle_joint
- removed joint kinova_right_robotiq_85_right_knuckle_joint
- removed joint left_back_wheel_joint
- removed joint left_front_wheel_joint
- removed joint right_back_wheel_joint
- removed joint right_front_wheel_joint
- added joint eddie_base_link_joint: type fixed, parent eddie_base_footprint, child eddie_base_link, origin xyz=0 0 0.2164 rpy=0 0 0
- added joint eddie_front_left_drive_attachment_joint: type fixed, parent eddie_base_link, child eddie_front_left_drive_attachment_link, origin xyz=0.2078 0.1880 -0.0632 rpy=0 0 1.5708
- added joint eddie_front_left_drive_l_wheel_joint: type fixed, parent eddie_front_left_drive_struct_link, child eddie_front_left_drive_l_wheel_link, origin xyz=0.0008 -0.0403 -0.0366 rpy=1.5708 3.1416 0, axis 0 0 1
- added joint eddie_front_left_drive_pivot_joint: type fixed, parent eddie_front_left_drive_attachment_link, child eddie_front_left_drive_struct_link, origin xyz=-0.0100 -0.0006 -0.0641 rpy=0 0 1.5708, axis 0 0 1
- added joint eddie_front_left_drive_r_wheel_joint: type fixed, parent eddie_front_left_drive_struct_link, child eddie_front_left_drive_r_wheel_link, origin xyz=0.0008 0.0407 -0.0366 rpy=-1.5708 0 0, axis 0 0 1
- added joint eddie_front_right_drive_attachment_joint: type fixed, parent eddie_base_link, child eddie_front_right_drive_attachment_link, origin xyz=0.2078 -0.1880 -0.0632 rpy=0 0 -1.5708
- added joint eddie_front_right_drive_l_wheel_joint: type fixed, parent eddie_front_right_drive_struct_link, child eddie_front_right_drive_l_wheel_link, origin xyz=0.0008 -0.0403 -0.0366 rpy=1.5708 3.1416 0, axis 0 0 1
- added joint eddie_front_right_drive_pivot_joint: type fixed, parent eddie_front_right_drive_attachment_link, child eddie_front_right_drive_struct_link, origin xyz=-0.0100 -0.0006 -0.0641 rpy=0 0 -1.5708, axis 0 0 1
- added joint eddie_front_right_drive_r_wheel_joint: type fixed, parent eddie_front_right_drive_struct_link, child eddie_front_right_drive_r_wheel_link, origin xyz=0.0008 0.0407 -0.0366 rpy=-1.5708 0 0, axis 0 0 1
- added joint eddie_front_right_laser_attachment_joint: type fixed, parent eddie_base_link, child eddie_front_right_laser_attachment_link, origin xyz=0.2193 -0.2391 0.0682 rpy=0 0 0
- added joint eddie_front_right_laser_joint: type fixed, parent eddie_front_right_laser_attachment_link, child eddie_front_right_laser_link, origin xyz=0 0 0 rpy=3.141592653589793 0 -0.7854
- added joint eddie_imu_joint: type fixed, parent eddie_base_link, child eddie_imu_link, origin xyz=0 0 0 rpy=0 0 0
- added joint eddie_left_arm_attachment_joint: type fixed, parent eddie_base_link, child eddie_left_arm_attachment_link, origin xyz=-0.1502 0.06789999999999999 0.5344 rpy=0 0.09 0.7925
- added joint eddie_left_arm_base_joint: type fixed, parent eddie_left_arm_attachment_link, child eddie_left_arm_base_link, origin xyz=0.01549 0 0 rpy=1.5708 -1.5708 1.5708
- added joint eddie_left_arm_camera_module: type fixed, parent eddie_left_arm_end_effector_link, child eddie_left_arm_camera_link, origin xyz=0 0.05639 -0.00305 rpy=3.141592653589793 3.141592653589793 0
- added joint eddie_left_arm_color_module: type fixed, parent eddie_left_arm_end_effector_link, child eddie_left_arm_camera_color_frame, origin xyz=0 0.05639 -0.00305 rpy=3.141592653589793 3.141592653589793 0
- added joint eddie_left_arm_depth_module: type fixed, parent eddie_left_arm_end_effector_link, child eddie_left_arm_camera_depth_frame, origin xyz=0.0275 0.066 -0.00305 rpy=3.141592653589793 3.141592653589793 0
- added joint eddie_left_arm_end_effector: type fixed, parent eddie_left_arm_bracelet_link, child eddie_left_arm_end_effector_link, origin xyz=0 0 -0.0615250000000001 rpy=3.14159265358979 1.09937075168372E-32 0, axis 0 0 0
- added joint eddie_left_arm_joint_1: type continuous, parent eddie_left_arm_base_link, child eddie_left_arm_shoulder_link, origin xyz=0 0 0.15643 rpy=3.1416 2.7629E-18 -4.9305E-36, axis 0 0 1, limit effort=39 velocity=1.3963
- added joint eddie_left_arm_joint_2: type revolute, parent eddie_left_arm_shoulder_link, child eddie_left_arm_half_arm_1_link, origin xyz=0 0.005375 -0.12838 rpy=1.5708 2.1343E-17 -1.1102E-16, axis 0 0 1, limit lower=-2.24 upper=2.24 effort=39 velocity=1.3963
- added joint eddie_left_arm_joint_3: type continuous, parent eddie_left_arm_half_arm_1_link, child eddie_left_arm_half_arm_2_link, origin xyz=0 -0.21038 -0.006375 rpy=-1.5708 1.2326E-32 -2.9122E-16, axis 0 0 1, limit effort=39 velocity=1.3963
- added joint eddie_left_arm_joint_4: type revolute, parent eddie_left_arm_half_arm_2_link, child eddie_left_arm_forearm_link, origin xyz=0 0.006375 -0.21038 rpy=1.5708 -6.6954E-17 -1.6653E-16, axis 0 0 1, limit lower=-2.57 upper=2.57 effort=39 velocity=1.3963
- added joint eddie_left_arm_joint_5: type continuous, parent eddie_left_arm_forearm_link, child eddie_left_arm_spherical_wrist_1_link, origin xyz=0 -0.20843 -0.006375 rpy=-1.5708 2.2204E-16 -6.373E-17, axis 0 0 1, limit effort=9 velocity=1.2218
- added joint eddie_left_arm_joint_6: type revolute, parent eddie_left_arm_spherical_wrist_1_link, child eddie_left_arm_spherical_wrist_2_link, origin xyz=0 0.00017505 -0.10593 rpy=1.5708 9.2076E-28 -8.2157E-15, axis 0 0 1, limit lower=-2.09 upper=2.09 effort=9 velocity=1.2218
- added joint eddie_left_arm_joint_7: type continuous, parent eddie_left_arm_spherical_wrist_2_link, child eddie_left_arm_bracelet_link, origin xyz=0 -0.10593 -0.00017505 rpy=-1.5708 -5.5511E-17 9.6396E-17, axis 0 0 1, limit effort=9 velocity=1.2218
- added joint eddie_left_arm_robotiq_85_base_joint: type fixed, parent eddie_left_arm_end_effector_link, child eddie_left_arm_robotiq_85_base_link, origin xyz=0 0 0.0 rpy=0 0 0
- added joint eddie_left_arm_robotiq_85_grasp_joint: type fixed, parent eddie_left_arm_robotiq_85_base_link, child eddie_left_arm_robotiq_85_grasp_link, origin xyz=0 0 0.1489 rpy=0 0 0
- added joint eddie_left_arm_robotiq_85_left_finger_joint: type fixed, parent eddie_left_arm_robotiq_85_left_knuckle_link, child eddie_left_arm_robotiq_85_left_finger_link, origin xyz=0.03152616 0.0 -0.00376347 rpy=0 0 0
- added joint eddie_left_arm_robotiq_85_left_finger_tip_joint: type continuous, parent eddie_left_arm_robotiq_85_left_finger_link, child eddie_left_arm_robotiq_85_left_finger_tip_link, origin xyz=0.00563134 0.0 0.04718515 rpy=0 0 0, axis 0 -1 0, mimic joint=eddie_left_arm_robotiq_85_left_knuckle_joint multiplier=-1
- added joint eddie_left_arm_robotiq_85_left_inner_knuckle_joint: type continuous, parent eddie_left_arm_robotiq_85_base_link, child eddie_left_arm_robotiq_85_left_inner_knuckle_link, origin xyz=0.0127 0.0 0.06142 rpy=0 0 0, axis 0 -1 0, mimic joint=eddie_left_arm_robotiq_85_left_knuckle_joint
- added joint eddie_left_arm_robotiq_85_left_knuckle_joint: type revolute, parent eddie_left_arm_robotiq_85_base_link, child eddie_left_arm_robotiq_85_left_knuckle_link, origin xyz=0.03060114 0.0 0.05490452 rpy=0 0 0, axis 0 -1 0, limit lower=0.0 upper=0.8 effort=50 velocity=0.5
- added joint eddie_left_arm_robotiq_85_right_finger_joint: type fixed, parent eddie_left_arm_robotiq_85_right_knuckle_link, child eddie_left_arm_robotiq_85_right_finger_link, origin xyz=-0.03152616 0.0 -0.00376347 rpy=0 0 0
- added joint eddie_left_arm_robotiq_85_right_finger_tip_joint: type continuous, parent eddie_left_arm_robotiq_85_right_finger_link, child eddie_left_arm_robotiq_85_right_finger_tip_link, origin xyz=-0.00563134 0.0 0.04718515 rpy=0 0 0, axis 0 -1 0, mimic joint=eddie_left_arm_robotiq_85_left_knuckle_joint
- added joint eddie_left_arm_robotiq_85_right_inner_knuckle_joint: type continuous, parent eddie_left_arm_robotiq_85_base_link, child eddie_left_arm_robotiq_85_right_inner_knuckle_link, origin xyz=-0.0127 0.0 0.06142 rpy=0 0 0, axis 0 -1 0, mimic joint=eddie_left_arm_robotiq_85_left_knuckle_joint multiplier=-1
- added joint eddie_left_arm_robotiq_85_right_knuckle_joint: type revolute, parent eddie_left_arm_robotiq_85_base_link, child eddie_left_arm_robotiq_85_right_knuckle_link, origin xyz=-0.03060114 0.0 0.05490452 rpy=0 0 0, axis 0 -1 0, limit lower=-0.8 upper=0.0 effort=50 velocity=0.5, mimic joint=eddie_left_arm_robotiq_85_left_knuckle_joint multiplier=-1
- added joint eddie_rear_left_drive_attachment_joint: type fixed, parent eddie_base_link, child eddie_rear_left_drive_attachment_link, origin xyz=-0.2078 0.1880 -0.0632 rpy=0 0 1.5708
- added joint eddie_rear_left_drive_l_wheel_joint: type fixed, parent eddie_rear_left_drive_struct_link, child eddie_rear_left_drive_l_wheel_link, origin xyz=0.0008 -0.0403 -0.0366 rpy=1.5708 3.1416 0, axis 0 0 1
- added joint eddie_rear_left_drive_pivot_joint: type fixed, parent eddie_rear_left_drive_attachment_link, child eddie_rear_left_drive_struct_link, origin xyz=-0.0100 -0.0006 -0.0641 rpy=0 0 1.5708, axis 0 0 1
- added joint eddie_rear_left_drive_r_wheel_joint: type fixed, parent eddie_rear_left_drive_struct_link, child eddie_rear_left_drive_r_wheel_link, origin xyz=0.0008 0.0407 -0.0366 rpy=-1.5708 0 0, axis 0 0 1
- added joint eddie_rear_left_laser_attachment_joint: type fixed, parent eddie_base_link, child eddie_rear_left_laser_attachment_link, origin xyz=-0.2193 0.2386 0.0682 rpy=0 0 0
- added joint eddie_rear_left_laser_joint: type fixed, parent eddie_rear_left_laser_attachment_link, child eddie_rear_left_laser_link, origin xyz=0 0 0 rpy=3.141592653589793 0 2.3562
- added joint eddie_rear_right_drive_attachment_joint: type fixed, parent eddie_base_link, child eddie_rear_right_drive_attachment_link, origin xyz=-0.2078 -0.1880 -0.0632 rpy=0 0 -1.5708
- added joint eddie_rear_right_drive_l_wheel_joint: type fixed, parent eddie_rear_right_drive_struct_link, child eddie_rear_right_drive_l_wheel_link, origin xyz=0.0008 -0.0403 -0.0366 rpy=1.5708 3.1416 0, axis 0 0 1
- added joint eddie_rear_right_drive_pivot_joint: type fixed, parent eddie_rear_right_drive_attachment_link, child eddie_rear_right_drive_struct_link, origin xyz=-0.0100 -0.0006 -0.0641 rpy=0 0 -1.5708, axis 0 0 1
- added joint eddie_rear_right_drive_r_wheel_joint: type fixed, parent eddie_rear_right_drive_struct_link, child eddie_rear_right_drive_r_wheel_link, origin xyz=0.0008 0.0407 -0.0366 rpy=-1.5708 0 0, axis 0 0 1
- added joint eddie_right_arm_attachment_joint: type fixed, parent eddie_base_link, child eddie_right_arm_attachment_link, origin xyz=-0.1502 -0.0673 0.5344 rpy=0 0.09 -0.7924
- added joint eddie_right_arm_base_joint: type fixed, parent eddie_right_arm_attachment_link, child eddie_right_arm_base_link, origin xyz=0.01549 0 0 rpy=1.5708 -1.5708 1.5708
- added joint eddie_right_arm_camera_module: type fixed, parent eddie_right_arm_end_effector_link, child eddie_right_arm_camera_link, origin xyz=0 0.05639 -0.00305 rpy=3.141592653589793 3.141592653589793 0
- added joint eddie_right_arm_color_module: type fixed, parent eddie_right_arm_end_effector_link, child eddie_right_arm_camera_color_frame, origin xyz=0 0.05639 -0.00305 rpy=3.141592653589793 3.141592653589793 0
- added joint eddie_right_arm_depth_module: type fixed, parent eddie_right_arm_end_effector_link, child eddie_right_arm_camera_depth_frame, origin xyz=0.0275 0.066 -0.00305 rpy=3.141592653589793 3.141592653589793 0
- added joint eddie_right_arm_end_effector: type fixed, parent eddie_right_arm_bracelet_link, child eddie_right_arm_end_effector_link, origin xyz=0 0 -0.0615250000000001 rpy=3.14159265358979 1.09937075168372E-32 0, axis 0 0 0
- added joint eddie_right_arm_ft_sensor_joint: type fixed, parent eddie_right_arm_end_effector_link, child eddie_right_arm_ft_sensor_link, origin xyz=0 0 0 rpy=0 0 0
- added joint eddie_right_arm_joint_1: type continuous, parent eddie_right_arm_base_link, child eddie_right_arm_shoulder_link, origin xyz=0 0 0.15643 rpy=3.1416 2.7629E-18 -4.9305E-36, axis 0 0 1, limit effort=39 velocity=1.3963
- added joint eddie_right_arm_joint_2: type revolute, parent eddie_right_arm_shoulder_link, child eddie_right_arm_half_arm_1_link, origin xyz=0 0.005375 -0.12838 rpy=1.5708 2.1343E-17 -1.1102E-16, axis 0 0 1, limit lower=-2.24 upper=2.24 effort=39 velocity=1.3963
- added joint eddie_right_arm_joint_3: type continuous, parent eddie_right_arm_half_arm_1_link, child eddie_right_arm_half_arm_2_link, origin xyz=0 -0.21038 -0.006375 rpy=-1.5708 1.2326E-32 -2.9122E-16, axis 0 0 1, limit effort=39 velocity=1.3963
- added joint eddie_right_arm_joint_4: type revolute, parent eddie_right_arm_half_arm_2_link, child eddie_right_arm_forearm_link, origin xyz=0 0.006375 -0.21038 rpy=1.5708 -6.6954E-17 -1.6653E-16, axis 0 0 1, limit lower=-2.57 upper=2.57 effort=39 velocity=1.3963
- added joint eddie_right_arm_joint_5: type continuous, parent eddie_right_arm_forearm_link, child eddie_right_arm_spherical_wrist_1_link, origin xyz=0 -0.20843 -0.006375 rpy=-1.5708 2.2204E-16 -6.373E-17, axis 0 0 1, limit effort=9 velocity=1.2218
- added joint eddie_right_arm_joint_6: type revolute, parent eddie_right_arm_spherical_wrist_1_link, child eddie_right_arm_spherical_wrist_2_link, origin xyz=0 0.00017505 -0.10593 rpy=1.5708 9.2076E-28 -8.2157E-15, axis 0 0 1, limit lower=-2.09 upper=2.09 effort=9 velocity=1.2218
- added joint eddie_right_arm_joint_7: type continuous, parent eddie_right_arm_spherical_wrist_2_link, child eddie_right_arm_bracelet_link, origin xyz=0 -0.10593 -0.00017505 rpy=-1.5708 -5.5511E-17 9.6396E-17, axis 0 0 1, limit effort=9 velocity=1.2218
- added joint eddie_right_arm_robotiq_85_base_joint: type fixed, parent eddie_right_arm_ft_sensor_link, child eddie_right_arm_robotiq_85_base_link, origin xyz=0 0 0.064 rpy=0 0 0
- added joint eddie_right_arm_robotiq_85_grasp_joint: type fixed, parent eddie_right_arm_robotiq_85_base_link, child eddie_right_arm_robotiq_85_grasp_link, origin xyz=0 0 0.1489 rpy=0 0 0
- added joint eddie_right_arm_robotiq_85_left_finger_joint: type fixed, parent eddie_right_arm_robotiq_85_left_knuckle_link, child eddie_right_arm_robotiq_85_left_finger_link, origin xyz=0.03152616 0.0 -0.00376347 rpy=0 0 0
- added joint eddie_right_arm_robotiq_85_left_finger_tip_joint: type continuous, parent eddie_right_arm_robotiq_85_left_finger_link, child eddie_right_arm_robotiq_85_left_finger_tip_link, origin xyz=0.00563134 0.0 0.04718515 rpy=0 0 0, axis 0 -1 0, mimic joint=eddie_right_arm_robotiq_85_left_knuckle_joint multiplier=-1
- added joint eddie_right_arm_robotiq_85_left_inner_knuckle_joint: type continuous, parent eddie_right_arm_robotiq_85_base_link, child eddie_right_arm_robotiq_85_left_inner_knuckle_link, origin xyz=0.0127 0.0 0.06142 rpy=0 0 0, axis 0 -1 0, mimic joint=eddie_right_arm_robotiq_85_left_knuckle_joint
- added joint eddie_right_arm_robotiq_85_left_knuckle_joint: type revolute, parent eddie_right_arm_robotiq_85_base_link, child eddie_right_arm_robotiq_85_left_knuckle_link, origin xyz=0.03060114 0.0 0.05490452 rpy=0 0 0, axis 0 -1 0, limit lower=0.0 upper=0.8 effort=50 velocity=0.5
- added joint eddie_right_arm_robotiq_85_right_finger_joint: type fixed, parent eddie_right_arm_robotiq_85_right_knuckle_link, child eddie_right_arm_robotiq_85_right_finger_link, origin xyz=-0.03152616 0.0 -0.00376347 rpy=0 0 0
- added joint eddie_right_arm_robotiq_85_right_finger_tip_joint: type continuous, parent eddie_right_arm_robotiq_85_right_finger_link, child eddie_right_arm_robotiq_85_right_finger_tip_link, origin xyz=-0.00563134 0.0 0.04718515 rpy=0 0 0, axis 0 -1 0, mimic joint=eddie_right_arm_robotiq_85_left_knuckle_joint
- added joint eddie_right_arm_robotiq_85_right_inner_knuckle_joint: type continuous, parent eddie_right_arm_robotiq_85_base_link, child eddie_right_arm_robotiq_85_right_inner_knuckle_link, origin xyz=-0.0127 0.0 0.06142 rpy=0 0 0, axis 0 -1 0, mimic joint=eddie_right_arm_robotiq_85_left_knuckle_joint multiplier=-1
- added joint eddie_right_arm_robotiq_85_right_knuckle_joint: type revolute, parent eddie_right_arm_robotiq_85_base_link, child eddie_right_arm_robotiq_85_right_knuckle_link, origin xyz=-0.03060114 0.0 0.05490452 rpy=0 0 0, axis 0 -1 0, limit lower=-0.8 upper=0.0 effort=50 velocity=0.5, mimic joint=eddie_right_arm_robotiq_85_left_knuckle_joint multiplier=-1
